Commit message: Rename robot from 'my_diffbot' to 'warehouse_bot'

File: my_diffbot.urdf.xacro (robot description, xacro)
@@ -1,5 +1,4 @@
 <?xml version="1.0"?>
-<robot xmlns:xacro="http://www.ros.org/wiki/xacro" name="my_diffbot">
-  <!-- Define properties for easy modification -->
+<robot xmlns:xacro="http://www.ros.org/wiki/xacro" name="warehouse_bot">
   <xacro:property name="base_width" value="0.4"/>
   <xacro:property name="base_length" value="0.6"/>
@@ -11,6 +10,5 @@
   <xacro:property name="lidar_radius" value="0.05"/>
   <xacro:property name="lidar_height" value="0.07"/>
-  <xacro:include filename="$(find robot_pkg)/urdf/my_diffbot.gazebo"/>
-  <!-- Base Link (Robot Body) -->
+  <xacro:include filename="$(find warehouse_pkg)/urdf/warehouse_bot.gazebo"/>
   <link name="base_link">
     <visual>
@@ -36,5 +34,4 @@
     </inertial>
   </link>
-  <!-- Base Footprint (for navigation) -->
   <link name="base_footprint"/>
   <joint name="base_footprint_joint" type="fixed">
@@ -43,5 +40,4 @@
     <origin xyz="0 0 ${wheel_radius}" rpy="0 0 0"/>
   </joint>
-<!-- Left Wheel -->
   <link name="left_wheel_link">
     <visual>
@@ -68,10 +64,9 @@
   </link>
   <joint name="left_wheel_joint" type="continuous">
-    <parent link="base_link"/>
-    <child link="left_wheel_link"/>
-    <origin xyz="${-base_length/4} ${wheel_separation/2} -0.07" rpy="0 0 0"/>
-    <axis xyz="0 1 0"/>
+   <parent link="base_link"/>
+   <child link="left_wheel_link"/>
+   <origin xyz="-0.1 ${wheel_separation/2} ${-base_height/2}" rpy="0 0 0"/>
+   <axis xyz="0 1 0"/>
   </joint>
-  <!-- Right Wheel -->
   <link name="right_wheel_link">
     <visual>
@@ -98,10 +93,9 @@
   </link>
   <joint name="right_wheel_joint" type="continuous">
-    <parent link="base_link"/>
-    <child link="right_wheel_link"/>
-    <origin xyz="${-base_length/4} ${-wheel_separation/2} -0.07" rpy="0 0 0"/>
-    <axis xyz="0 1 0"/>
+   <parent link="base_link"/>
+   <child link="right_wheel_link"/>
+   <origin xyz="-0.1 ${-wheel_separation/2} ${-base_height/2}" rpy="0 0 0"/>
+   <axis xyz="0 1 0"/>
   </joint>
-  <!-- Caster Wheel (front support) -->
   <link name="caster_link">
     <visual>
@@ -132,5 +126,4 @@
     <origin xyz="${base_length/2 - caster_radius} 0 ${-base_height/2 - caster_radius/2}" rpy="0 0 0"/>
   </joint>
-<!-- LIDAR Sensor -->
   <link name="lidar_link">
     <visual>
